Commit message: Mise à jour de la configuration du robot quadrupède : ajout des joints et des interfaces pour ros2_control, et intégration du plugin Gazebo.

File: src/quadruped_description/quadruped/robot.urdf (robot description, URDF)
Before this commit: robot quadruped_robot, 14 links, 13 joints
Links:
- added link dummy_root, mass 0.001
Joints:
- added joint dummy_to_body: type fixed, parent dummy_root, child body, origin xyz=0 0 0 rpy=0 0 0

Commit message: Mise à jour du modèle URDF : simplification du lien racine et ajustement de la configuration du plugin Gazebo pour ros2_control.

File: src/quadruped_description/quadruped/robot.urdf (robot description, URDF)
Before this commit: robot quadruped_robot, 15 links, 14 joints
Links:
- link dummy_root: mass 0.001 -> None
